File: Hardware/V3S-devboard-module/DIMM.kicad_sch (KiCad schematic)
At the start: 3 parts, among them J1 Bus_DDR4_Edge_Conn

Commit message: schematic improvements
Parts:
- removed R1: R_US, Resistor_SMD:R_0402_1005Metric_Pad0.72x0.64mm_HandSolder, symbol Device:R_US
- J1: footprint SODIMM-DDR4:Bus_DDR4_Conn_Edge -> lpddr4-testbed-footprints:Bus_DDR4_Conn_Edge
Connections:
- net LCD_D4: now also J1.125; no longer J1.11
- net LCD_D20: now reaches J1.101
- net LCD_D19: now reaches J1.103
- net LCD_D18: now reaches J1.105
- net LCD_D15: now reaches J1.107
- net LCD_D14: now reaches J1.109
- net LCD_D13: now reaches J1.111
- net LCD_D12: now reaches J1.113
- net LCD_D11: now reaches J1.115
- net LCD_D10: now reaches J1.117
- net LCD_D7: now reaches J1.119
- net LCD_D6: now reaches J1.121
- net LCD_D5: now reaches J1.123
- net LCD_D3: now reaches J1.127
- net LCD_D2: now reaches J1.129
- net LCD_D23: now reaches J1.95
- net LCD_D22: now reaches J1.97
- net LCD_D21: now reaches J1.99
Other:
- moved on the sheet: A1B, J1A
