File: Hardware/V3S-devboard-module/uP.kicad_sch (KiCad schematic)
At the start: 1 part, among them U1 V3S

Commit message: minor changes
Parts:
- added R8: 6K, symbol Device:R_Small_US
Connections:
- net VDD_CPU: now reaches U1.38 (VDD-CPU4)
- net VDD_CPU: now also U1.47 (VDD-CPU5), U1.51 (VDD-CPU6), U1.56 (VDD-CPU7)
- net VCC_IO: now reaches U1.50 (VCC-IO3)
- net VCC_IO: now also U1.57 (VCC-IO2)
- net PC0_SPI_MISO: now reaches U1.52 (PC0/SDC2_CLK/SPI_MISO)
- net PC1_SPI_CLK: now reaches U1.53 (PC1/SDC2_CMD/SPI_CLK)
- net PC2_SPI_CS: now reaches U1.54 (PC2/SDC2_RST/SPI_CS)
- net PC3_SPI_MOSI: now reaches U1.55 (PC3/SDC2_D0/SPI_MOSI)
- net VDD_SYS: now reaches U1.58 (VDD-SYS4)
- net VDD_SYS: now also U1.64 (VDD-SYS5), U1.80 (VDD-SYS0)
- net VCC_DRAM: now reaches U1.59 (VCC-DRAM8)
- net VCC_DRAM: now also U1.60 (VCC-DRAM9), U1.61 (VCC-DRAM10), U1.62 (VCC-DARM11), U1.65 (VCC-DRAM0), U1.66 (VCC-DRAM1), U1.67 (VCC-DRAM2), U1.68 (VCC-DRAM3), U1.69 (VCC-DRAM4), U1.70 (VCC-DRAM5), U1.72 (VCC-DRAM6)
- net SVREF: now reaches U1.63 (SVREF1)
- net SVREF: now also U1.71 (SVREF0)
- net SZQ: now reaches U1.73 (SZQ)
- net X24MOUT: now reaches U1.74 (X24MOUT)
- net X24_MIN: now reaches U1.75 (X24MIN)
- net ETH_LED_LINK: now reaches U1.77 (EPHY-LINK-LED)
- net ETH_LED_SPD: now reaches U1.78 (EPHY-SPD-LED)
- net MSCI_D0_P: now reaches U1.81 (MCSI-D0P)
- net MSCI_D0_N: now reaches U1.82 (MCSI-D0N)
- net MSCI_D1_P: now reaches U1.83 (MCSI-D1P)
- net MSCI_D1_N: now reaches U1.84 (MCSI-D1N)
- net VCC_MSCI: now reaches U1.85 (VCC-MCSI)
- net MSCI_CLK_P: now reaches U1.86 (MCSI-CKP)
- net MSCI_CLK_N: now reaches U1.87 (MCSI-CKN)
- net VDD_PHY: now reaches U1.88 (EPHY-VDD)
- net ETH_RX_N: now reaches U1.89 (EPHY-RXN)
- net ETH_RX_P: now reaches U1.90 (EPHY-RXP)
- net ETH_TX_N: now reaches U1.91 (EPHY-TXN)
- net ETH_TX_P: now reaches U1.92 (EPHY-TXP)
- net VCC_PHY: now reaches U1.93 (EPHY-VCC)
- net at U1.94 (EPHY-RTX): now also R8.1
- new net GND: R8.2
Other:
- note added: "DRAM"
- note added: "EPHY"
- note added: "MIPI"
- note added: "SYS"

Commit message: more shcematic
Parts:
- added C10, C11, C12, C13: 18p, symbol Device:C_Small
- added R10, R9: 10M, symbol Device:R_Small_US
- added R11: 240, symbol Device:R_Small_US
- added Y1: Crystal_GND23_Small, symbol Device:Crystal_GND23_Small
- added Y2: Crystal_GND23_Small, Crystal:Crystal_SMD_3225-4Pin_3.2x2.5mm, symbol Device:Crystal_GND23_Small
Connections:
- net GND: now also C10.1, C11.1, C12.1, C13.1, R11.2, Y1.2, Y1.3, Y2.2, Y2.3
- net SZQ: now also R11.1
- net VCC_IO: now also U1.104 (VCC-IO0), U1.127 (VCC-IO1)
- net VDD_CPU: now also U1.20 (VDD-CPU3), U1.21 (VDD-CPU2), U1.25 (VDD-CPU1), U1.26 (VDD-CPU0)
- net VDD_SYS: now also U1.108 (VDD-SYS1), U1.126 (VDD-SYS2), U1.19 (VDD-SYS3)
- net X24_MIN: now also C12.2, R10.1, Y2.1
- net PG4_SDCI_D2: now reaches U1.1 (PG4/SDC1_D2/PG_EINT4)
- net PE20_MCSI_MCLK: now reaches U1.10 (PE20/CSI_FIELD/CSI_MIPI_MCLK)
- net VCC_USB: now reaches U1.109 (VCC-USB)
- net PE19_LCD_D21: now reaches U1.11 (PE19/CSI_D15/LCD_D21)
- net USB_N: now reaches U1.110 (USB-DN)
- net USB_P: now reaches U1.111 (USB-DP)
- net HBIAS: now reaches U1.119 (HBIAS)
- net VCC_PE: now reaches U1.12 (VCC-PE0)
- net VCC_PE: now also U1.29 (VCC-PE1)
- net HPOUTR: now reaches U1.120 (HPOUTR)
- net HPOUTL: now reaches U1.121 (HPOUTL)
- net HPCOMFB: now reaches U1.124 (HPCOMFB)
- net HPCOM: now reaches U1.125 (HPCOM)
- net PG5_SDCI_D3: now reaches U1.128 (PG5/SDC1_D3/PG_EINT5)
- net PE18_LCD_D20: now reaches U1.13 (PE18/CSI_D14/LCD_D20)
- net PE17_LCD_D19: now reaches U1.14 (PE17/CSI_D13/LCD_D19)
- net PE16_LCD_D18: now reaches U1.15 (PE16/CSI_D12/LCD_D18)
- net PE15_LCD_D15: now reaches U1.16 (PE15/CSI_D11/LCD_D15)
- net PE14_LCD_D14: now reaches U1.17 (PE14/CSI_D10/LCD_D14)
- net PE13_LCD_D13: now reaches U1.18 (PE13/CSI_D9/LCD_D13)
- net PG3_SDCI_D1: now reaches U1.2 (PG3/SDC1_D1/PG_EINT3)
- net PE12_LCD_D12: now reaches U1.22 (PE12/CSI_D8/LCD_D12)
- net PE11_LCD_D11: now reaches U1.23 (PE11/CSI_D7/LCD_D11)
- net PE10_LCD_D10: now reaches U1.24 (PE10/CSI_D6/LCD_D10)
- net PE8_LCD_D7: now reaches U1.27 (PE9/CSI_D5/LCD_D7)
- net PE8_LCD_D6: now reaches U1.28 (PE8/CSI_D4/LCD_D6)
- net PG2_SDCI_D0: now reaches U1.3 (PG2/SDC1_D0/PG_EINT2)
- net PE7_LCD_D5: now reaches U1.30 (PE7/CSI_D3/LCD_D5)
- net PE6_LCD_D4: now reaches U1.31 (PE6/CSI_D2/LCD_D4)
- net PE5_LCD_D3: now reaches U1.32 (PE5/CSI_D1/LCD_D3)
- net PE4_LCD_D2: now reaches U1.33 (PE4/CSI_D0/LCD_D2)
- net PE3_LCD_VSYNC: now reaches U1.34 (PE3/CSI_VSYNC/LCD_VSYNC)
- net PE2_LCD_HSYNC: now reaches U1.35 (PE2/CSI_HSYNC/LCD_HSYNC)
- net PE1_LCD_DE: now reaches U1.36 (PE1/CSI_MCLK/LCD_DE)
- net PE0_LCD_CLK: now reaches U1.37 (PE0/CSI_PCLK/LCD_CLK)
- net PB0_UART2TX: now reaches U1.39 (PB0/UART2_TX/PB_EINT0)
- net PG0_MCSI_PDWN: now reaches U1.4 (PG1/SDC1_CMD/PG_EINT1)
- net PB1_UART2RX: now reaches U1.40 (PB1/UART2_RX/PB_EINT1)
- net PB2_UART2RTS: now reaches U1.41 (PB2/UART2_RTS/PB_EINT2)
- net PB3_UART2CTS: now reaches U1.42 (PB3/UART2_CTS/PB_EINT3)
- net PB4_PWM0: now reaches U1.43 (PB4/PWM0/PB_EINT4)
- net PB5_PWM1: now reaches U1.44 (PB5/PWM1/PB_EINT5)
- net PB6_SCK: now reaches U1.45 (PB6/TWI0_SCK/PB_EINT6)
- net PB7_SDA: now reaches U1.46 (PB7/TWI0_SDA/PB_EINT7)
- net PB8_SCK_UART0TX: now reaches U1.48 (PB8/TWI1_SCK/UART0_TX/PB_EINT8)
- net PB9_SDA_UART0RX: now reaches U1.49 (PB9/TWI1_SDA/UART0_RX/PB_EINT9)
- net PG0_MCSI_RST: now reaches U1.5 (PG0/SDC1_CLK/PG_EINT0)
- net PE24_LCD_D23: now reaches U1.6 (PE24/LCD_D23)
- net PE23_LCD_D22: now reaches U1.7 (PE23/LCD_D22)
- net PE22_CSI_SDA: now reaches U1.8 (PE22/CSI_SDA/TWI1_SDA/UART1_RX)
- net PE21_CSI_SCK: now reaches U1.9 (PE21/CSI_SCK/TWI1_SCK/UART1_TX)
- net X32KOUT: now reaches U1.95 (X32KOUT)
- net X32KOUT: now also C11.2, R9.2, Y1.4
- net X32KIN: now reaches U1.96 (X32KIN)
- net X32KIN: now also C10.2, R9.1, Y1.1
- net RESET: now reaches U1.99 (RESET)
- new net: C13.2, R10.2, Y2.4
Other:
- note added: "check pinout! 3225"
- note added: "check pinout! MC-146"

Commit message: more schematic changes
Connections:
- net AVCC: now also U1.115 (AVCC)
- net GND: now also U1.116 (AGND)
- net VCC_DRAM: now also U1.79 (VCC-DRAM7)
- net VCC_PLL: now also U1.76 (VCC-PLL)
- net PF6: now reaches U1.100 (PF6)
- net PF5_SDC0D2_JTAGCK1: now reaches U1.101 (F5/SDC0_D2/JTAG_CK1)
- net PF4_SDC0D3_UART0RX: now reaches U1.102 (PF4/SDC0_D3/UART0_RX)
- net PF3_SDC0CMD_JTAGDO1: now reaches U1.103 (PF3/SDC0_CMD/JTAG_DO1)
- net PF2_SDC0CLK_UART0TX: now reaches U1.105 (PF2/SDC0_CLK/UART0_TX)
- net PF1_SDC0D0_JTAGDI1: now reaches U1.106 (PF1/SDC0_D0/JTAG_DI1)
- net PF0_SDC0D1_JTAGDI1: now reaches U1.107 (PF0/SDC0_D1/JTAG_MS1)
- net LRADC0: now reaches U1.112 (LRADC0)
- net MCIN1_P: now reaches U1.113 (MICIN1P)
- net MCIN1_N: now reaches U1.114 (MICIN1N)
- net VRA1: now reaches U1.117 (VRA1)
- net VRA2: now reaches U1.118 (VRA2)
- net VCC_HP: now reaches U1.122 (HPVCCIN)
- net VCC_HP_BP: now reaches U1.123 (HPVCCBP)
- net VCC_RTCIO: now reaches U1.97 (RTC-VIO)
- net VCC_RTC: now reaches U1.98 (VCC-RTC)
- net ETH_RX_N renamed ETH0.RX_N
- net ETH_RX_P renamed ETH0.RX_P
- net ETH_TX_N renamed ETH0.TX_N
- net ETH_TX_P renamed ETH0.TX_P
Other:
- moved on the sheet: R8, U1

Commit message: schematic work
Connections:
- net PB0_UART2TX renamed UART2.TX
- net PB1_UART2RX renamed UART2.RX
- net PB2_UART2RTS renamed UART2.RTS
- net PB3_UART2CTS renamed UART2.CTS
- net PB8_SCK_UART0TX renamed UART0.TX
- net PB9_SDA_UART0RX renamed UART0.RX
- net PC0_SPI_MISO renamed SPI.MISO
- net PC1_SPI_CLK renamed SPI.CLK
- net PC2_SPI_CS renamed SPI.CS
- net PC3_SPI_MOSI renamed SPI.MOSI
- net PE0_LCD_CLK renamed LCD0.CLK
- net PE10_LCD_D10 renamed LCD_D10
- net PE11_LCD_D11 renamed LCD_D11
- net PE12_LCD_D12 renamed LCD_D12
- net PE13_LCD_D13 renamed LCD_D13
- net PE14_LCD_D14 renamed LCD_D14
- net PE15_LCD_D15 renamed LCD_D15
- net PE16_LCD_D18 renamed LCD_D18
- net PE17_LCD_D19 renamed LCD_D19
- net PE18_LCD_D20 renamed LCD_D20
- net PE19_LCD_D21 renamed LCD_D21
- net PE1_LCD_DE renamed LCD0.DE
- net PE23_LCD_D22 renamed LCD_D22
- net PE24_LCD_D23 renamed LCD_D23
- net PE2_LCD_HSYNC renamed LCD0.HSYNC
- net PE3_LCD_VSYNC renamed LCD0.VSYNC
- net PE4_LCD_D2 renamed LCD_D2
- net PE5_LCD_D3 renamed LCD_D3
- net PE6_LCD_D4 renamed LCD_D4
- net PE7_LCD_D5 renamed LCD_D5
- net PE8_LCD_D6 renamed LCD_D6
- net PE8_LCD_D7 renamed LCD_D7
