File: Hardware/V3S-devboard-module/uP.kicad_sch (KiCad schematic)
At the start: 29 parts, among them J201 Micro_SD_Card_Det1, SW201 SW_MEC_5E, U201 V3S, U202 W25Q128JVS, Y201 Crystal_GND24_Small, Y202 Crystal_GND24_Small

Commit message: more tests
Parts:
- removed R205: 10M, Resistor_SMD:R_0402_1005Metric, symbol Device:R_Small_US
- removed Y201: Crystal_GND24_Small, Crystal:Crystal_SMD_2520-4Pin_2.5x2.0mm, symbol Device:Crystal_GND24_Small
- added R301: 100K, Resistor_SMD:R_0402_1005Metric, symbol Device:R_Small_US
- added Y201: Crystal_Small, Crystal:Crystal_SMD_3215-2Pin_3.2x1.5mm, symbol Device:Crystal_Small
- R218, R219: footprint Resistor_SMD:R_0603_1608Metric -> Resistor_SMD:R_0402_1005Metric
Connections:
- net AVCC: now also R301.1
- net LRADC0: now also R301.2
- net X32KIN: now also Y201.1
- net X32KOUT: now also Y201.2
- net HBIAS renamed ADCDAC.HBIAS
- net HPCOM renamed ADCDAC.HPCOM
- net HPCOMFB renamed ADCDAC.HPCOMFB
- net HPOUTL renamed ADCDAC.HPOUTL
- net HPOUTR renamed ADCDAC.HPOUTR
- net MCIN1_N renamed ADCDAC.MIC_N
- net MCIN1_P renamed ADCDAC.MIC_P
Other:
- note added: "2-32.768KHz 9pF 20ppm at least 40ppm C2848222"
- note added: "check pinout! 3225 CRY-TSX3225 24M-20pF-10PPM at least 50ppm"
- note removed: "2-32.768KHz 9pF 20ppm"
- note removed: "check pinout! 3225 CRY-TSX3225"

Commit message: more layout
Parts:
- removed R216, R217: 33, Resistor_SMD:R_0603_1608Metric, symbol Device:R_Small_US
- added CN1: AS0BC21-S30BE-7H, v3s-devboard-module:CONN-SMD_AS0BC21-S30BE-7H, symbol v3s-devboard-module:AS0BC21-S30BE-7H
- C235: footprint Capacitor_SMD:C_0603_1608Metric -> Capacitor_SMD:C_0402_1005Metric
- R208, R220: footprint Resistor_SMD:R_0603_1608Metric -> Resistor_SMD:R_0402_1005Metric

Commit message: layout
Connections:
- net PB2 is gone; now on net USB.USB_ID: U201.41 (PB2/UART2_RTS/PB_EINT2)
- net USB.USB_ID: no longer U201.100 (PF6)
- net PF6 renamed SD_DET
- net SD_DET: now also U201.100 (PF6)
Changed lines of the file:
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@@
 	)
 	(bus_entry
-		(at 190.5 68.58)
-		(size 2.54 2.54)
+		(at 137.16 240.03)
+		(size 2.54 -2.54)
 		(stroke
 			(width 0)
@@
 	(wire
 		(pts
+			(xy 193.04 69.85) (xy 193.04 83.82)
+		)
+		(stroke
+			(width 0)
+			(type default)
+		)
+	)
+	(wire
+		(pts
 			(xy 359.41 54.61) (xy 367.03 54.61)
 		)
@@
 	(bus
 		(pts
+			(xy 138.43 241.3) (xy 138.43 256.54)
+		)
+		(stroke
+			(width 0)
+			(type default)
+		)
+	)
+	(bus
+		(pts
 			(xy 52.07 116.84) (xy 52.07 119.38)
 		)
@@
 	(bus
 		(pts
-			(xy 134.62 240.03) (xy 139.7 240.03)
+			(xy 36.83 24.13) (xy 58.42 24.13)
 		)
 		(stroke
@@
 		)
 	)
-	(bus
+	(wire
 		(pts
-			(xy 36.83 24.13) (xy 58.42 24.13)
+			(xy 339.09 151.13) (xy 350.52 151.13)
 		)
 		(stroke
@@
 	(wire
 		(pts
-			(xy 339.09 151.13) (xy 350.52 151.13)
+			(xy 139.7 215.9) (xy 139.7 237.49)
 		)
 		(stroke
@@
 	(wire
 		(pts
-			(xy 139.7 215.9) (xy 139.7 231.14)
-		)
-		(stroke
-			(width 0)
-			(type default)
-		)
-	)
-	(wire
-		(pts
 			(xy 313.69 236.22) (xy 313.69 241.3)
 		)
@@
 	(bus
 		(pts
-			(xy 189.23 67.31) (xy 189.23 57.15)
-		)
-		(stroke
-			(width 0)
-			(type default)
-		)
-	)
-	(bus
-		(pts
 			(xy 168.91 241.3) (xy 170.18 240.03)
 		)
@@
 	(wire
 		(pts
-			(xy 193.04 71.12) (xy 193.04 83.82)
-		)
-		(stroke
-			(width 0)
-			(type default)
-		)
-	)
-	(wire
-		(pts
 			(xy 54.61 172.72) (xy 76.2 172.72)
 		)
@@
 	(bus
 		(pts
-			(xy 189.23 67.31) (xy 190.5 68.58)
-		)
-		(stroke
-			(width 0)
-			(type default)
-		)
-	)
-	(bus
-		(pts
 			(xy 50.8 168.91) (xy 52.07 170.18)
 		)
@@
 	(bus
 		(pts
+			(xy 135.89 241.3) (xy 135.89 251.46)
+		)
+		(stroke
+			(width 0)
+			(type default)
+		)
+	)
+	(bus
+		(pts
 			(xy 52.07 111.76) (xy 52.07 114.3)
 		)
@@
 		)
 	)
+	(bus
+		(pts
+			(xy 138.43 241.3) (xy 139.7 240.03)
+		)
+		(stroke
+			(width 0)
+			(type default)
+		)
+	)
 	(wire
 		(pts
@@
 		)
 	)
+	(bus
+		(pts
+			(xy 135.89 241.3) (xy 137.16 240.03)
+		)
+		(stroke
+			(width 0)
+			(type default)
+		)
+	)
 	(wire
 		(pts
@@
 		)
 	)
-	(label "USB{USB}"
-		(at 189.23 57.15 270)
-		(fields_autoplaced yes)
-		(effects
-			(font
-				(size 1.27 1.27)
-			)
-			(justify right bottom)
-		)
-	)
 	(label "CSI.MCSI_MCLK"
 		(at 54.61 142.24 0)
@@
 		)
 	)
-	(label "PF6"
+	(label "SD_DET"
 		(at 313.69 241.3 90)
 		(fields_autoplaced yes)
@@
 		)
 	)
-	(label "PF6"
+	(label "SD_DET"
 		(at 304.8 214.63 0)
 		(fields_autoplaced yes)
@@
 		)
 	)
-	(label "PB2"
-		(at 139.7 231.14 90)
-		(fields_autoplaced yes)
-		(effects
-			(font
-				(size 1.27 1.27)
-			)
-			(justify left bottom)
-		)
-	)
 	(label "LRADC0"
 		(at 38.1 66.04 0)
@@
 		)
 	)
+	(label "USB{USB}"
+		(at 135.89 251.46 90)
+		(fields_autoplaced yes)
+		(effects
+			(font
+				(size 1.27 1.27)
+			)
+			(justify left bottom)
+		)
+	)
 	(label "SDC0.CMD"
 		(at 304.8 196.85 0)
@@
 		)
 	)
+	(label "UART2{UART}"
+		(at 138.43 256.54 90)
+		(fields_autoplaced yes)
+		(effects
+			(font
+				(size 1.27 1.27)
+			)
+			(justify left bottom)
+		)
+	)
 	(label "PF3_SDC0CMD_JTAGDO1"
 		(at 322.58 241.3 0)
@@
 		)
 	)
+	(label "USB.USB_ID"
+		(at 139.7 224.79 270)
+		(fields_autoplaced yes)
+		(effects
+			(font
+				(size 1.27 1.27)
+			)
+			(justify right bottom)
+		)
+	)
 	(label "LCD_D4"
 		(at 54.61 195.58 0)
@@
 		)
 	)
+	(label "SD_DET"
+		(at 193.04 77.47 90)
+		(fields_autoplaced yes)
+		(effects
+			(font
+				(size 1.27 1.27)
+			)
+			(justify left bottom)
+		)
+	)
 	(label "LCD_D11"
 		(at 54.61 175.26 0)
@@
 		(fields_autoplaced yes)
 		(effects
-			(font
-				(size 1.27 1.27)
-			)
-			(justify left bottom)
-		)
-	)
-	(label "USB.USB_ID"
-		(at 193.04 83.82 90)
-		(fields_autoplaced yes)
-		(effects

Commit message: layout
Parts:
- removed SW201: SW_MEC_5E, v3s-devboard-module:SW_SKRPACE010, symbol Switch:SW_MEC_5E
- R207: footprint Resistor_SMD:R_0603_1608Metric -> Resistor_SMD:R_0402_1005Metric
Other:
- moved on the sheet: C234
Changed lines of the file:
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@@
 	)
 	(junction
-		(at 350.52 85.09)
-		(diameter 0)
-		(color 0 0 0 0)
-	)
-	(junction
 		(at 372.11 30.48)
 		(diameter 0)
@@
 	)
 	(junction
-		(at 360.68 85.09)
-		(diameter 0)
-		(color 0 0 0 0)
-	)
-	(junction
-		(at 350.52 87.63)
-		(diameter 0)
-		(color 0 0 0 0)
-	)
-	(junction
 		(at 180.34 215.9)
 		(diameter 0)
@@
 	)
 	(junction
+		(at 350.52 85.09)
+		(diameter 0)
+		(color 0 0 0 0)
+	)
+	(junction
 		(at 350.52 33.02)
 		(diameter 0)
@@
 		)
 	)
-	(wire
-		(pts
-			(xy 360.68 85.09) (xy 363.22 85.09)
-		)
-		(stroke
-			(width 0)
-			(type default)
-		)
-	)
 	(bus
 		(pts
@@
 	(wire
 		(pts
-			(xy 350.52 87.63) (xy 350.52 97.79)
-		)
-		(stroke
-			(width 0)
-			(type default)
-		)
-	)
-	(wire
-		(pts
 			(xy 195.58 215.9) (xy 198.12 215.9)
 		)
@@
 		)
 	)
-	(wire
-		(pts
-			(xy 360.68 85.09) (xy 360.68 87.63)
-		)
-		(stroke
-			(width 0)
-			(type default)
-		)
-	)
 	(bus
 		(pts
@@
 	(wire
 		(pts
-			(xy 350.52 85.09) (xy 350.52 87.63)
+			(xy 350.52 85.09) (xy 350.52 97.79)
 		)
 		(stroke
@@
 	(wire
 		(pts
-			(xy 353.06 87.63) (xy 350.52 87.63)
+			(xy 353.06 85.09) (xy 350.52 85.09)
 		)
 		(stroke
@@
 	(wire
 		(pts
-			(xy 358.14 87.63) (xy 360.68 87.63)
+			(xy 358.14 85.09) (xy 363.22 85.09)
 		)
 		(stroke
@@
 		)
 	)
+	(wire
+		(pts
+			(xy 49.53 92.71) (xy 36.83 92.71)
+		)
+		(stroke
+			(width 0)
+			(type default)
+		)
+	)
 	(bus
 		(pts
@@
 		)
 	)
+	(label "RESET"
+		(at 36.83 92.71 0)
+		(fields_autoplaced yes)
+		(effects
+			(font
+				(size 1.27 1.27)
+			)
+			(justify left bottom)
+		)
+	)
 	(label "ADCDAC.HPCOM"
 		(at 124.46 80.01 90)
@@
 		)
 	)
+	(global_label "RESET"
+		(shape input)
+		(at 36.83 92.71 180)
+		(fields_autoplaced yes)
+		(effects
+			(font
+				(size 1.27 1.27)
+			)
+			(justify right)
+		)
+		(property "Intersheetrefs" "${INTERSHEET_REFS}"
+			(at 25.5596 92.71 0)
+			(effects
+				(font
+					(size 1.27 1.27)
+				)
+				(justify right)
+				(hide yes)
+			)
+		)
+	)
 	(global_label "LCD_D[0..23]"
 		(shape input)
@@
 	(symbol
 		(lib_id "Device:C_Small")
-		(at 355.6 87.63 270)
+		(at 355.6 85.09 270)
 		(unit 1)
 		(exclude_from_sim no)
@@
 		(dnp no)
 		(property "Reference" "C234"
-			(at 355.6 90.932 90)
+			(at 355.6 88.392 90)
 			(effects
 				(font
@@
 		)
 		(property "Value" "1u"
-			(at 355.6 93.472 90)
+			(at 355.6 90.932 90)
 			(effects
 				(font
@@
 		)
 		(property "Footprint" "Capacitor_SMD:C_0603_1608Metric"
-			(at 355.6 87.63 0)
+			(at 355.6 85.09 0)
 			(effects
 				(font
@@
 		)
 		(property "Datasheet" "~"
-			(at 355.6 87.63 0)
+			(at 355.6 85.09 0)
 			(effects
 				(font
@@
 		)
 		(property "Description" "Unpolarized capacitor, small symbol"
-			(at 355.6 87.63 0)
+			(at 355.6 85.09 0)
 			(effects
 				(font
@@
 			)
 		)
-		(property "Footprint" "Resistor_SMD:R_0603_1608Metric"
+		(property "Footprint" "Resistor_SMD:R_0402_1005Metric"
 			(at 345.44 85.09 0)
 			(effects
@@
 					(unit 1)
 				)
-			)
-		)
-	)
-	(symbol
-		(lib_id "Switch:SW_MEC_5E")
-		(at 355.6 85.09 0)
-		(unit 1)
-		(exclude_from_sim no)
-		(in_bom yes)
-		(on_board yes)
-		(dnp no)
-		(fields_autoplaced yes)
-		(property "Reference" "SW201"
-			(at 355.6 77.47 0)
-			(effects
-				(font
-					(size 1.27 1.27)
-				)
-			)
-		)
-		(property "Value" "SW_MEC_5E"
-			(at 354.33 86.36 90)
-			(effects
-				(font
-					(size 1.27 1.27)
-				)
-				(justify right)
-				(hide yes)
-			)
-		)
-		(property "Footprint" "v3s-devboard-module:SW_SKRPACE010"
-			(at 355.6 77.47 0)
-			(effects
-				(font
-					(size 1.27 1.27)
-				)
-				(hide yes)
-			)
-		)
-		(property "Datasheet" "http://www.apem.com/int/index.php?controller=attachment&id_attachment=1371"
-			(at 355.6 77.47 0)
-			(effects
-				(font
-					(size 1.27 1.27)
-				)
-				(hide yes)
-			)
-		)
-		(property "Description" "MEC 5E single pole normally-open tactile switch"
-			(at 355.6 85.09 0)
-			(effects
-				(font
-					(size 1.27 1.27)
-				)
-				(hide yes)
-			)
-		)
-		(pin "1"
-		)
-		(pin "2"
-		)
-		(pin "3"
-		)
-		(pin "4"
-		)
-		(instances
-			(project "V3S-devboard-module"
-				(path "/5d41c08e-2331-42df-a2d5-1aeb6ed4388c/f51f2d23-c28c-4ea4-895a-4b3207c38b48"
-					(reference "SW201")
-					(unit 1)
-				)

Commit message: layout
Parts:
- removed R211, R212, R213, R214, R215: 10k, Resistor_SMD:R_0603_1608Metric, symbol Device:R_Small_US
- added C7: 1n, Capacitor_SMD:C_0402_1005Metric, symbol Device:C_Small
- added R7: 10k, Resistor_SMD:R_0402_1005Metric, symbol Device:R_Small_US
- added R8: 0, Resistor_SMD:R_0402_1005Metric, symbol Device:R_Small_US
- added RN1: R_Pack04, Resistor_SMD:R_Array_Concave_4x0402, symbol Device:R_Pack04
- added SW1: SW_MEC_5E, v3s-devboard-module:SW_SKRPACE010, symbol Switch:SW_MEC_5E
- C234: value 1u -> 100n; footprint Capacitor_SMD:C_0603_1608Metric -> Capacitor_SMD:C_0402_1005Metric
- R210: footprint Resistor_SMD:R_0603_1608Metric -> Resistor_SMD:R_0402_1005Metric
Connections:
- net 3V3: now also R7.2, RN1.5 (R4.2), RN1.6 (R3.2), RN1.7 (R2.2), RN1.8 (R1.2)
- net GND: now also C7.1, R8.1, SW1.3 (K), SW1.4 (A)
- net LRADC0: now also C7.2
- net SDC0.CMD: now also RN1.2 (R2.1)
- net SDC0.D0: now also R7.1
- net SDC0.D1: now also RN1.1 (R1.1)
- net SDC0.D2: now also RN1.4 (R4.1)
- net SDC0.D3: now also RN1.3 (R3.1)
- net SPI.MISO: now also R8.2, SW1.1, SW1.2

Commit message: layout
Parts:
- removed CN1: AS0BC21-S30BE-7H, v3s-devboard-module:CONN-SMD_AS0BC21-S30BE-7H, symbol v3s-devboard-module:AS0BC21-S30BE-7H
- J201: LCSC (none) -> C7529389
- SW1: LCSC (none) -> C139797
- U201: LCSC (none) -> C2687449; LCSC Part C2687449 -> (none)
- U202: LCSC (none) -> C97521
- Y201: LCSC (none) -> C2848222
Changed lines of the file:
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@@
 			)
 		)
+		(property "LCSC" "C2848222"
+			(at 345.44 30.48 90)
+			(effects
+				(font
+					(size 1.27 1.27)
+				)
+				(hide yes)
+			)
+		)
 		(pin "1"
 		)
@@
 			)
 		)
+		(property "LCSC" "C139797"
+			(at 336.55 172.72 0)
+			(effects
+				(font
+					(size 1.27 1.27)
+				)
+				(hide yes)
+			)
+		)
 		(pin "2"
 		)
@@
 			)
 		)
-		(property "LCSC Part" "C2687449"
+		(property "LCSC" "C2687449"
 			(at 149.86 226.06 0)
 			(effects
@@
 			)
 		)
+		(property "LCSC" "C7529389"
+			(at 370.84 201.93 0)
+			(effects
+				(font
+					(size 1.27 1.27)
+				)
+				(hide yes)
+			)
+		)
 		(pin "1"
 		)
@@
 	)
 	(symbol
-		(lib_id "v3s-devboard-module:AS0BC21-S30BE-7H")
-		(at 139.7 345.44 90)
-		(unit 1)
-		(exclude_from_sim no)
-		(in_bom yes)
-		(on_board yes)
-		(dnp no)
-		(fields_autoplaced yes)
-		(property "Reference" "CN1"
-			(at 93.98 344.1699 90)
-			(effects
-				(font
-					(size 1.27 1.27)
-				)
-				(justify left)
-			)
-		)
-		(property "Value" "AS0BC21-S30BE-7H"
-			(at 93.98 346.7099 90)
-			(effects
-				(font
-					(size 1.27 1.27)
-				)
-				(justify left)
-			)
-		)
-		(property "Footprint" "v3s-devboard-module:CONN-SMD_AS0BC21-S30BE-7H"
-			(at 194.31 345.44 0)
-			(effects
-				(font
-					(size 1.27 1.27)
-				)
-				(hide yes)
-			)
-		)
-		(property "Datasheet" ""
-			(at 139.7 345.44 0)
-			(effects
-				(font
-					(size 1.27 1.27)
-				)
-				(hide yes)
-			)
-		)
-		(property "Description" ""
-			(at 139.7 345.44 0)
-			(effects
-				(font
-					(size 1.27 1.27)
-				)
-				(hide yes)
-			)
-		)
-		(property "LCSC Part" "C3020019"
-			(at 196.85 345.44 0)
-			(effects
-				(font
-					(size 1.27 1.27)
-				)
-				(hide yes)
-			)
-		)
-		(pin "37"
-		)
-		(pin "65"
-		)
-		(pin "21"
-		)
-		(pin "5"
-		)
-		(pin "66"
-		)
-		(pin "68"
-		)
-		(pin "69"
-		)
-		(pin "34"
-		)
-		(pin "67"
-		)
-		(pin "7"
-		)
-		(pin "42"
-		)
-		(pin "58"
-		)
-		(pin "17"
-		)
-		(pin "71"
-		)
-		(pin "12"
-		)
-		(pin "59"
-		)
-		(pin "46"
-		)
-		(pin "55"
-		)
-		(pin "52"
-		)
-		(pin "22"
-		)
-		(pin "70"
-		)
-		(pin "49"
-		)
-		(pin "72"
-		)
-		(pin "73"
-		)
-		(pin "74"
-		)
-		(pin "14"
-		)
-		(pin "18"
-		)
-		(pin "23"
-		)
-		(pin "43"
-		)
-		(pin "3"
-		)
-		(pin "1"
-		)
-		(pin "20"
-		)
-		(pin "11"
-		)
-		(pin "19"
-		)
-		(pin "50"
-		)
-		(pin "2"
-		)
-		(pin "53"
-		)
-		(pin "36"
-		)
-		(pin "39"
-		)
-		(pin "41"
-		)
-		(pin "54"
-		)
-		(pin "35"
-		)
-		(pin "13"
-		)
-		(pin "57"
-		)
-		(pin "61"
-		)
-		(pin "16"
-		)
-		(pin "62"
-		)
-		(pin "6"
-		)
-		(pin "10"
-		)
-		(pin "32"
-		)
-		(pin "33"
-		)
-		(pin "45"
-		)
-		(pin "44"
-		)
-		(pin "63"
-		)
-		(pin "48"
-		)
-		(pin "15"
-		)
-		(pin "4"
-		)
-		(pin "38"
-		)
-		(pin "51"
-		)
-		(pin "60"
-		)
-		(pin "40"
-		)
-		(pin "47"
-		)
-		(pin "56"
-		)
-		(pin "64"
-		)
-		(pin "8"
-		)
-		(pin "9"
-		)
-		(pin "77"
-		)
-		(pin "75"
-		)
-		(pin "76"
-		)
-		(instances
-			(project "V3S-devboard-module"
-				(path "/5d41c08e-2331-42df-a2d5-1aeb6ed4388c/f51f2d23-c28c-4ea4-895a-4b3207c38b48"
-					(reference "CN1")
-					(unit 1)
-				)
-			)
-		)
-	)
-	(symbol
 		(lib_id "Memory_Flash:W25Q128JVS")
 		(at 360.68 153.67 0)
@@
 			(at 360.68 153.67 0)
 			(effects
+				(font
+					(size 1.27 1.27)
+				)
+				(hide yes)
+			)
+		)
+		(property "LCSC" "C97521"
+			(at 360.68 153.67 0)
+			(effects

Commit message: re-annotated everything
Parts:
- renumbered C7 to C235, C235 to C236, R206 to R205, R207 to R206, R220 to R207, R301 to R208, R208 to R209, R8 to R210, R209 to R211, R219 to R212, R218 to R213, R210 to R214, R7 to R215, RN1 to RN201, SW1 to SW201

Commit message: pre production tests
Parts:
- C230, C231, C232, C233: LCSC (none) -> C541431
- C234, C236: LCSC (none) -> C1525
- C235: value 1n -> 100n; LCSC (none) -> C1525
- R204: LCSC (none) -> C138067
- R205: LCSC (none) -> C114755
- R206: LCSC (none) -> C93943; Precision (none) -> 1%
- R207: footprint Resistor_SMD:R_0402_1005Metric -> Resistor_SMD:R_0805_2012Metric; LCSC (none) -> C2828725
- R208: LCSC (none) -> C60491
- R209, R215: LCSC (none) -> C60490
- R210: LCSC (none) -> C106231; now fitted
- R211: footprint Resistor_SMD:R_0603_1608Metric -> Resistor_SMD:R_0402_1005Metric; LCSC (none) -> C138002
- R212, R213: LCSC (none) -> C138002; Precision (none) -> 1%
- R214: LCSC (none) -> C93943
- RN201: LCSC (none) -> C1736647
- Y202: LCSC (none) -> C15643
Changed lines of the file:
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@@
 	(wire
 		(pts
+			(xy 392.43 214.63) (xy 391.16 214.63)
+		)
+		(stroke
+			(width 0)
+			(type default)
+		)
+	)
+	(wire
+		(pts
 			(xy 185.42 69.85) (xy 185.42 83.82)
 		)
@@
 			)
 		)
-		(property "Precision" ""
+		(property "Precision" "1%"
 			(at 159.766 229.362 90)
 			(effects
@@
 			)
 		)
+		(property "LCSC" "C138002"
+			(at 157.48 233.68 90)
+			(effects
+				(font
+					(size 1.27 1.27)
+				)
+				(hide yes)
+			)
+		)
 		(pin "2"
 		)
@@
 			)
 		)
+		(property "LCSC" "C15643"
+			(at 345.44 52.07 90)
+			(effects
+				(font
+					(size 1.27 1.27)
+				)
+				(hide yes)
+			)
+		)
 		(pin "2"
 		)
@@
 			)
 		)
+		(property "LCSC" "C1525"
+			(at 377.19 140.97 0)
+			(effects
+				(font
+					(size 1.27 1.27)
+				)
+				(hide yes)
+			)
+		)
 		(pin "1"
 		)
@@
 			)
 		)
-		(property "Precision" ""
+		(property "Precision" "1%"
 			(at 162.306 224.282 90)
 			(effects
@@
 			)
 		)
+		(property "LCSC" "C138002"
+			(at 160.02 228.6 90)
+			(effects
+				(font
+					(size 1.27 1.27)
+				)
+				(hide yes)
+			)
+		)
 		(pin "2"
 		)
@@
 			)
 		)
+		(property "LCSC" "C541431"
+			(at 369.57 54.61 90)
+			(effects
+				(font
+					(size 1.27 1.27)
+				)
+				(hide yes)
+			)
+		)
 		(pin "1"
 		)
@@
 			)
 		)
+		(property "LCSC" "C1736647"
+			(at 370.84 234.95 0)
+			(effects
+				(font
+					(size 1.27 1.27)
+				)
+				(hide yes)
+			)
+		)
 		(pin "6"
 		)
@@
 			)
 		)
-		(property "Footprint" "Resistor_SMD:R_0402_1005Metric"
+		(property "Footprint" "Resistor_SMD:R_0805_2012Metric"
 			(at 226.06 104.14 0)
 			(effects
@@
 			)
 		)
+		(property "LCSC" "C2828725"
+			(at 226.06 104.14 90)
+			(effects
+				(font
+					(size 1.27 1.27)
+				)
+				(hide yes)
+			)
+		)
 		(pin "2"
 		)
@@
 			)
 		)
-		(property "Value" "1n"
+		(property "Value" "100n"
 			(at 359.41 121.412 90)
 			(effects
@@
 			)
 		)
+		(property "LCSC" "C1525"
+			(at 359.41 115.57 90)
+			(effects
+				(font
+					(size 1.27 1.27)
+				)
+				(hide yes)
+			)
+		)
 		(pin "1"
 		)
@@
 			)
 		)
-		(property "Footprint" "Resistor_SMD:R_0603_1608Metric"
+		(property "Footprint" "Resistor_SMD:R_0402_1005Metric"
 			(at 331.47 201.93 0)
 			(effects
@@
 			)
 		)
+		(property "LCSC" "C138002"
+			(at 331.47 201.93 90)
+			(effects
+				(font
+					(size 1.27 1.27)
+				)
+				(hide yes)
+			)
+		)
 		(pin "2"
 		)
@@
 		(in_bom yes)
 		(on_board yes)
-		(dnp yes)
+		(dnp no)
 		(property "Reference" "R210"
 			(at 337.8201 175.26 0)
@@
 			)
 		)
+		(property "LCSC" "C106231"
+			(at 336.55 172.72 0)
+			(effects
+				(font
+					(size 1.27 1.27)
+				)
+				(hide yes)
+			)
+		)
 		(pin "2"
 		)
@@
 			)
 		)
+		(property "LCSC" "C541431"
+			(at 369.57 27.94 90)
+			(effects
+				(font
+					(size 1.27 1.27)
+				)
+				(hide yes)
+			)
+		)
 		(pin "1"
 		)
@@
 			)
 		)
+		(property "LCSC" "C541431"
+			(at 369.57 49.53 90)
+			(effects
+				(font
+					(size 1.27 1.27)
+				)
+				(hide yes)
+			)
+		)
 		(pin "1"
 		)
@@
 			)
 		)
+		(property "LCSC" "C1525"
+			(at 355.6 85.09 90)
+			(effects
+				(font
+					(size 1.27 1.27)
+				)
+				(hide yes)
+			)
+		)
 		(pin "1"
 		)
@@
 			)
 		)
-		(property "Precision" ""
+		(property "Precision" "1%"
 			(at 349.758 87.376 90)
 			(effects
@@
 			)
 		)
+		(property "LCSC" "C93943"
+			(at 345.44 85.09 90)
+			(effects
+				(font
+					(size 1.27 1.27)
+				)
+				(hide yes)
+			)
+		)
 		(pin "2"
 		)
@@
 			)
 		)
+		(property "LCSC" "C60490"
+			(at 360.68 234.95 0)
+			(effects
+				(font
+					(size 1.27 1.27)
+				)
+				(hide yes)
+			)
+		)
 		(pin "2"
 		)
@@
 	(symbol
 		(lib_id "power:GND")
-		(at 391.16 214.63 0)
+		(at 392.43 214.63 0)
 		(unit 1)
 		(exclude_from_sim no)
@@
 		(dnp no)
 		(property "Reference" "#PWR0250"
-			(at 391.16 220.98 0)
+			(at 392.43 220.98 0)
 			(effects
 				(font
@@
 		)
 		(property "Value" "GND"
-			(at 391.414 217.932 90)
+			(at 392.684 217.932 90)
 			(effects
 				(font
@@
 		)
 		(property "Footprint" ""
-			(at 391.16 214.63 0)
+			(at 392.43 214.63 0)
 			(effects
 				(font
@@
 		)
 		(property "Datasheet" ""
-			(at 391.16 214.63 0)
+			(at 392.43 214.63 0)
 			(effects
 				(font
@@
 		)
 		(property "Description" "Power symbol creates a global label with name \"GND\" , ground"
-			(at 391.16 214.63 0)
+			(at 392.43 214.63 0)
 			(effects
 				(font
@@
 			)
 		)
+		(property "LCSC" "C60491"
+			(at 354.33 107.95 90)
+			(effects
+				(font
+					(size 1.27 1.27)
+				)
+				(hide yes)
+			)
+		)
 		(pin "2"
 		)
@@
 			)
 		)
+		(property "LCSC" "C541431"
+			(at 369.57 33.02 90)
+			(effects
+				(font
+					(size 1.27 1.27)
+				)
+				(hide yes)
+			)
+		)
 		(pin "1"
 		)
@@
 			)
 		)
+		(property "LCSC" "C60490"
+			(at 347.98 139.7 0)
+			(effects
+				(font
+					(size 1.27 1.27)
+				)
+				(hide yes)
+			)
+		)
 		(pin "2"
 		)
@@
 			)
 		)
+		(property "LCSC" "C93943"
+			(at 313.69 233.68 0)
+			(effects
+				(font
+					(size 1.27 1.27)
+				)
+				(hide yes)
+			)
+		)
 		(pin "2"
 		)
@@
 			)
 		)
+		(property "LCSC" "C138067"
+			(at 359.41 30.48 0)
+			(effects
+				(font
+					(size 1.27 1.27)
+				)
+				(hide yes)
+			)
+		)
 		(pin "2"
 		)
@@
 			)
 		)
+		(property "LCSC" "C114755"
+			(at 355.6 71.12 90)
+			(effects
+				(font
+					(size 1.27 1.27)
+				)
+				(hide yes)
+			)
+		)
