File: Hardware/V3S-devboard-module/V3S-devboard-module.kicad_pcb (KiCad board)
At the start: 2 copper layers, 22 x 4 mm, 88 parts, among them J201 Micro_SD_Card_Det1, J301 AS0BC21-S30BE-7H, SW201 SW_MEC_5E, U101 EA3036C, U102 XC6206PxxxMR, U201 V3S, U202 W25Q128JVS, Y201 Crystal_GND23_Small, Y202 Crystal_GND23_Small

Commit message: some layout
Parts:
- removed NT1: NetTie_2, NetTie:NetTie-2_SMD_Pad2.0mm
- added C1: 18p, Capacitor_SMD:C_0402_1005Metric, F.Cu at (8.79, 5.50)
- added C2: 10u, Capacitor_SMD:C_0603_1608Metric, F.Cu at (9.37, 0.76)
- added C3: 18p, Capacitor_SMD:C_0402_1005Metric, F.Cu at (8.79, 7.47)
- added C4: 10u, Capacitor_SMD:C_0603_1608Metric, F.Cu at (9.37, 3.27)
- added L1: 2.2u, Inductor_SMD:L_1008_2520Metric, F.Cu at (4.88, 1.38)
- added L2: 2.2u, Inductor_SMD:L_1008_2520Metric, F.Cu at (4.88, 5.12)
- added NT10: NetTie_2, NetTie:NetTie-2_SMD_Pad0.5mm, F.Cu at (184.9, 19.8)
- added NT11: NetTie_2, NetTie:NetTie-2_SMD_Pad0.5mm, F.Cu at (248.8, 75.7)
- added NT12: NetTie_2, NetTie:NetTie-2_SMD_Pad0.5mm, F.Cu at (184.9, 22.8)
- added NT13: NetTie_2, NetTie:NetTie-2_SMD_Pad0.5mm, F.Cu at (184.9, 24.3)
- added NT2: NetTie_2, NetTie:NetTie-2_SMD_Pad0.5mm, F.Cu at (215.5, 60.2)
- added NT3: NetTie_2, NetTie:NetTie-2_SMD_Pad0.5mm, F.Cu at (179.9, 21.3)
- added NT4: NetTie_2, NetTie:NetTie-2_SMD_Pad0.5mm, F.Cu at (179.9, 22.8)
- added NT5: NetTie_2, NetTie:NetTie-2_SMD_Pad0.5mm, F.Cu at (179.9, 24.3)
- added NT6: NetTie_2, NetTie:NetTie-2_SMD_Pad0.5mm, F.Cu at (182.4, 19.8)
- added NT7: NetTie_2, NetTie:NetTie-2_SMD_Pad0.5mm, F.Cu at (182.4, 21.3)
- added NT8: NetTie_2, NetTie:NetTie-2_SMD_Pad0.5mm, F.Cu at (182.4, 22.8)
- added NT9: NetTie_2, NetTie:NetTie-2_SMD_Pad0.5mm, F.Cu at (182.4, 24.3)
- added R1: 200K, Resistor_SMD:R_0402_1005Metric, F.Cu at (0.95, 0.49)
- added R2: 100K, Resistor_SMD:R_0402_1005Metric, F.Cu at (0.95, 2.48)
- added R3: 150K, Resistor_SMD:R_0402_1005Metric, F.Cu at (0.95, 4.47)
- added R4: 150K, Resistor_SMD:R_0402_1005Metric, F.Cu at (0.95, 6.46)
- C203, C204, C205, C206, C207, C208, C209, C210, C211, C212, C213, C214, C215, C216, C217, C218, C219: moved to B.Cu
- C220, C221, C227, C228: moved to F.Cu
- moved C223 106.0 mm to (244.1, 74.2), turned to 180 degrees
- moved REF** 83.0 mm to (223.4, 96.9), turned to 180 degrees
- moved U201 82.0 mm to (223.5, 69.1), turned to -90 degrees
- moved C204 81.6 mm to (222.9, 71.4), turned to -90 degrees
- moved C205 79.5 mm to (225.3, 71.8), turned to -90 degrees
- moved C203 78.7 mm to (221.3, 71.4), turned to -90 degrees
- moved C207 77.5 mm to (224.2, 71.8), turned to -90 degrees
- moved C206 75.9 mm to (219.7, 71.4), turned to -90 degrees
- moved C214 74.0 mm to (217.9, 70.2), turned to 180 degrees
- moved C215 73.6 mm to (217.9, 71.2), turned to 180 degrees
- moved C212 69.5 mm to (218.0, 67.3), turned to 180 degrees
- moved C213 69.1 mm to (218.0, 68.8), turned to 180 degrees
- moved R220 68.6 mm to (204.1, 56.1)
- moved C218 67.0 mm to (224.3, 66.8), turned to 90 degrees
- moved C219 65.0 mm to (223.2, 66.8), turned to 90 degrees
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Connections:
- C105 pad 1: Net-(U101-FB1) -> Net-(U101-FB3)
- C107 pad 1: Net-(U101-FB3) -> Net-(U101-FB1)
- C208 pad 2: 1V2 -> VDD_SYS
- C209 pad 2: 1V2 -> VDD_SYS
- C210 pad 2: 1V2 -> VDD_SYS
- C211 pad 2: 1V2 -> VDD_SYS
- C212 pad 2: 1V2 -> VDD_CPU
- C213 pad 2: 1V2 -> VDD_CPU
- C214 pad 2: 1V2 -> VDD_CPU
- C215 pad 2: 1V2 -> VDD_CPU
- C216 pad 2: 3V3 -> VCC_IO
- C217 pad 2: 3V3 -> VCC_IO
- C218 pad 2: 3V3 -> VCC_IO
- C219 pad 2: 3V3 -> VCC_IO
- C220 pad 2: 3V3 -> VCC_USB
- C221 pad 2: 3V3 -> VCC_MSCI
- C223 pad 2: 3V0 -> VCC_PLL
- C224 pad 2: 3V3 -> VCC_HP
- L101 pad 1: Net-(U101-LX1) -> Net-(U101-LX2)
- L102 pad 1: Net-(U101-LX2) -> Net-(U101-LX1)
- R101 pad 2: Net-(U101-FB1) -> Net-(U101-FB3)
- R102 pad 1: Net-(U101-FB1) -> Net-(U101-FB3)
- R103 pad 2: Net-(U101-FB3) -> Net-(U101-FB1)
- R104 pad 1: Net-(U101-FB3) -> Net-(U101-FB1)
- U201 pad 104: 3V3 -> VCC_IO
- U201 pad 108: 1V2 -> VDD_SYS
- U201 pad 109: 3V3 -> VCC_USB
- U201 pad 115: 3V0 -> AVCC
- U201 pad 12: 3V3 -> VCC_PE
- U201 pad 122: 3V3 -> VCC_HP
- U201 pad 126: 1V2 -> VDD_SYS
- U201 pad 127: 3V3 -> VCC_IO
- U201 pad 19: 1V2 -> VDD_SYS
- U201 pad 20: 1V2 -> VDD_CPU
- U201 pad 21: 1V2 -> VDD_CPU
- U201 pad 25: 1V2 -> VDD_CPU
- U201 pad 26: 1V2 -> VDD_CPU
- U201 pad 29: 3V3 -> VCC_PE
- U201 pad 38: 1V2 -> VDD_CPU
- U201 pad 47: 1V2 -> VDD_CPU
- U201 pad 50: 3V3 -> VCC_IO
- U201 pad 51: 1V2 -> VDD_CPU
- U201 pad 56: 1V2 -> VDD_CPU
- U201 pad 57: 3V3 -> VCC_IO
- U201 pad 58: 1V2 -> VDD_SYS
- U201 pad 64: 1V2 -> VDD_SYS
- U201 pad 76: 3V0 -> VCC_PLL
- U201 pad 80: 1V2 -> VDD_SYS
- U201 pad 85: 3V3 -> VCC_MSCI
- U201 pad 88: 1V2 -> VDD_PHY
- U201 pad 93: 3V3 -> VCC_PHY
Routing:
- net VDD_SYS: track 0.00 -> 72.4 mm, vias 0 -> 6
- net VCC_IO: track 0.00 -> 52.7 mm, vias 0 -> 10
- net VDD_CPU: track 0.00 -> 40.3 mm, vias 0 -> 1
- net VCC_DRAM: track 39.7 -> 54.0 mm, vias 0 -> 1
Other:
- board size 22 x 4 mm -> 26.2 x 52.8 mm
