File: Hardware/V3S-devboard-module/ext_conn.kicad_sch (KiCad schematic)
At the start: 1 part, among them CN2 AS0BC21-S30BE-7H

Commit message: general improvements. power almost complete
Parts:
- removed CN2: AS0BC21-S30BE-7H, v3s-devboard-module:CONN-SMD_AS0BC21-S30BE-7H, symbol v3s-devboard-module:AS0BC21-S30BE-7H
- added CN3: AS0BC21-S30BE-7H, v3s-devboard-module:m2-padKeyE, symbol v3s-devboard-module:m2-KeyE
Connections:
- net CSI.CSI_SCK: now also CN3.38
- net CSI.CSI_SDA: now also CN3.36
- net CSI.MCSI_CK_N: now also CN3.42
- net CSI.MCSI_CK_P: now also CN3.44
- net CSI.MCSI_D0_N: now also CN3.50
- net CSI.MCSI_D0_P: now also CN3.52
- net CSI.MCSI_D1_N: now also CN3.46
- net CSI.MCSI_D1_P: now also CN3.48
- net CSI.MCSI_MCLK: now also CN3.40
- net ETH0.RX_N: now also CN3.37
- net ETH0.RX_P: now also CN3.35
- net ETH0.TX_N: now also CN3.33
- net ETH0.TX_P: now also CN3.23
- net LCD0.CLK: now also CN3.34
- net LCD0.DE: now also CN3.32
- net LCD0.HSYNC: now also CN3.22
- net LCD0.VSYNC: now also CN3.20
- net LCD_D10: now also CN3.6
- net LCD_D11: now also CN3.4
- net LCD_D12: now also CN3.2
- net LCD_D13: now also CN3.17
- net LCD_D14: now also CN3.15
- net LCD_D15: now also CN3.13
- net LCD_D18: now also CN3.11
- net LCD_D19: now also CN3.9
- net LCD_D2: now also CN3.18
- net LCD_D20: now also CN3.7
- net LCD_D21: now also CN3.5
- net LCD_D22: now also CN3.3
- net LCD_D23: now also CN3.1
- net LCD_D3: now also CN3.16
- net LCD_D4: now also CN3.14
- net LCD_D5: now also CN3.12
- net LCD_D6: now also CN3.10
- net LCD_D7: now also CN3.8
- net SPI.CLK: now also CN3.43
- net SPI.CS: now also CN3.45
- net SPI.MISO: now also CN3.41
- net SPI.MOSI: now also CN3.47
- net UART0.RX: now also CN3.56
- net UART0.TX: now also CN3.54
- net UART2.CTS: now also CN3.53
- net UART2.RX: now also CN3.51
- net UART2.TX: now also CN3.49
- new net ETH_LED_LINK: CN3.21
- new net ETH_LED_SPD: CN3.19
Other:
- title: (none) -> Power

Commit message: fixed minor schematic issues
Parts:
- renumbered CN3 to J301
Connections:
- net USB.USB_P: now reaches J301.58
- net USB.USB_N: now reaches J301.60
- net SDC1.D2: now reaches J301.62
- net SDC1.D1: now reaches J301.64
- net SDC1.D0: now reaches J301.66
- net SDC1.CMD: now reaches J301.68
- net SDC1.CLK: now reaches J301.70

Commit message: some layout
Connections:
- net CSI.CSI_SCK: no longer J301.38
- net CSI.CSI_SDA: no longer J301.36
- net CSI.MCSI_CK_N: no longer J301.42
- net CSI.MCSI_CK_P: no longer J301.44
- net CSI.MCSI_D0_N: no longer J301.50
- net CSI.MCSI_D0_P: no longer J301.52
- net CSI.MCSI_D1_N: no longer J301.46
- net CSI.MCSI_D1_P: no longer J301.48
- net CSI.MCSI_MCLK: no longer J301.40
- net ETH0.RX_N: no longer J301.37
- net ETH0.RX_P: no longer J301.35
- net ETH0.TX_N: no longer J301.33
- net ETH0.TX_P: no longer J301.23
- net ETH_LED_LINK: no longer J301.21
- net ETH_LED_SPD: no longer J301.19
- net LCD0.CLK: no longer J301.34
- net LCD0.DE: no longer J301.32
- net LCD0.HSYNC: no longer J301.22
- net LCD0.VSYNC: no longer J301.20
- net LCD_D10: no longer J301.6
- net LCD_D11: no longer J301.4
- net LCD_D12: no longer J301.2
- net LCD_D13: no longer J301.17
- net LCD_D14: no longer J301.15
- net LCD_D15: no longer J301.13
- net LCD_D18: no longer J301.11
- net LCD_D19: no longer J301.9
- net LCD_D2: no longer J301.18
- net LCD_D20: no longer J301.7
- net LCD_D21: no longer J301.5
- net LCD_D22: no longer J301.3
- net LCD_D23: no longer J301.1
- net LCD_D3: no longer J301.16
- net LCD_D4: no longer J301.14
- net LCD_D5: no longer J301.12
- net LCD_D6: no longer J301.10
- net LCD_D7: no longer J301.8
- net SDC1.CLK: no longer J301.70
- net SDC1.CMD: no longer J301.68
- net SDC1.D0: no longer J301.66
- net SDC1.D1: no longer J301.64
- net SDC1.D2: no longer J301.62
- net UART0.RX: no longer J301.56
- net UART0.TX: no longer J301.54
- net USB.USB_N: no longer J301.60
- net USB.USB_P: no longer J301.58
- new net 5V: J301.1, J301.2, J301.3, J301.4
- new net GND: J301.5, J301.6, J301.7, J301.8

Commit message: layout testing
Connections:
- net CSI.CSI_SCK: now also J301.47
- net CSI.CSI_SDA: now also J301.48
- net CSI.MCSI_CK_N: now also J301.42
- net CSI.MCSI_CK_P: now also J301.44
- net CSI.MCSI_D0_N: now also J301.39
- net CSI.MCSI_D0_P: now also J301.41
- net CSI.MCSI_D1_N: now also J301.43
- net CSI.MCSI_D1_P: now also J301.45
- net CSI.MCSI_MCLK: now also J301.46
- net LCD_D10: now also J301.55
- net LCD_D11: now also J301.58
- net LCD_D12: now also J301.57
- net LCD_D13: now also J301.60
- net LCD_D14: now also J301.59
- net LCD_D15: now also J301.62
- net LCD_D18: now also J301.61
- net LCD_D19: now also J301.64
- net LCD_D2: now also J301.49
- net LCD_D20: now also J301.63
- net LCD_D21: now also J301.66
- net LCD_D22: now also J301.65
- net LCD_D23: now also J301.68
- net LCD_D3: now also J301.52
- net LCD_D4: now also J301.51
- net LCD_D5: now also J301.54
- net LCD_D6: now also J301.53
- net LCD_D7: now also J301.56
- net SDC1.CLK: now also J301.67
- net SDC1.CMD: now also J301.70
- net SDC1.D0: now also J301.69
- net SDC1.D1: now also J301.72
- net SDC1.D2: now also J301.71
- net SPI.CLK: no longer J301.43
- net SPI.CS: no longer J301.45
- net SPI.MISO: no longer J301.41
- net SPI.MOSI: no longer J301.47
- net UART2.CTS: no longer J301.53
- net UART2.RX: no longer J301.51
- net UART2.TX: no longer J301.49
- net USB.USB_N: now also J301.75
- net USB.USB_P: now also J301.73

Commit message: more layout testing
Connections:
- net CSI.MCSI_D0_N: now also J301.43; no longer J301.39
- net CSI.MCSI_D0_P: now also J301.45; no longer J301.41
- net CSI.MCSI_D1_N: now also J301.39; no longer J301.43
- net CSI.MCSI_D1_P: now also J301.41; no longer J301.45
- net ETH0.RX_N: now also J301.35
- net ETH0.RX_P: now also J301.33
- net ETH0.TX_N: now also J301.34
- net ETH0.TX_P: now also J301.32
- net LCD0.CLK: now also J301.36
- net LCD0.DE: now also J301.37
- net LCD0.HSYNC: now also J301.38
- net LCD0.VSYNC: now also J301.40

Commit message: more tests
Connections:
- net 5V: no longer J301.2, J301.4
- net GND: now also J301.2, J301.4; no longer J301.5, J301.6, J301.7, J301.8
- net PB6_SCK: now reaches J301.20
- net PB7_SDA: now reaches J301.22
- net USB.USB_ID: now reaches J301.74
Other:
- moved on the sheet: J301

Commit message: more layout
Connections:
- net LRADC0: now also J301.20
- net PB6_SCK: now also J301.19; no longer J301.20
- net PB7_SDA: now also J301.18; no longer J301.22
- net UART0.RX: now also J301.16
- net UART0.TX: now also J301.17
- net UART2.CTS: now also J301.21
- net UART2.RX: now also J301.22
- net UART2.TX: now also J301.23
Other:
- note added: "AS0BC21-S40BB-7H"

Commit message: layout
Connections:
- net 5V: now also J301.5
- net ADCDAC.HBIAS: now also J301.11
- net ADCDAC.HPCOM: now also J301.7
- net ADCDAC.HPCOMFB: now also J301.8
- net ADCDAC.HPOUTL: now also J301.9
- net ADCDAC.HPOUTR: now also J301.10
- net ETH_LED_LINK: now also J301.15
- net ETH_LED_SPD: now also J301.14
- net PB4_PWM0: now also J301.12
- net PB5_PWM1: now also J301.13
- net RESET: now reaches J301.6
