File: Hardware/V3S-devboard-module/ext_conn.kicad_sch (KiCad schematic)
At the start: 1 part, among them J301 AS0BC21-S30BE-7H

Commit message: layout
Changed lines of the file:
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@@
-	)
-	(bus_entry
-		(at 124.46 62.23)
-		(size 2.54 2.54)
-		(stroke
-			(width 0)
-			(type default)
-		)
 	)
 	(bus_entry
@@
 	)
 	(bus_entry
-		(at 124.46 64.77)
-		(size 2.54 2.54)
-		(stroke
-			(width 0)
-			(type default)
-		)
-	)
-	(bus_entry
 		(at 137.16 154.94)
 		(size -2.54 2.54)
@@
 	)
 	(bus_entry
-		(at 124.46 59.69)
-		(size 2.54 2.54)
-		(stroke
-			(width 0)
-			(type default)
-		)
-	)
-	(bus_entry
 		(at 73.66 137.16)
 		(size 2.54 2.54)
@@
 	)
 	(bus_entry
-		(at 124.46 57.15)
-		(size 2.54 2.54)
-		(stroke
-			(width 0)
-			(type default)
-		)
-	)
-	(bus_entry
 		(at 73.66 129.54)
 		(size 2.54 2.54)
@@
 	)
 	(bus_entry
-		(at 124.46 67.31)
-		(size 2.54 2.54)
-		(stroke
-			(width 0)
-			(type default)
-		)
-	)
-	(bus_entry
 		(at 137.16 144.78)
 		(size -2.54 2.54)
@@
 		)
 	)
-	(wire
-		(pts
-			(xy 127 64.77) (xy 148.59 64.77)
-		)
-		(stroke
-			(width 0)
-			(type default)
-		)
-	)
 	(bus
 		(pts
@@
 	(wire
 		(pts
-			(xy 127 67.31) (xy 148.59 67.31)
-		)
-		(stroke
-			(width 0)
-			(type default)
-		)
-	)
-	(wire
-		(pts
 			(xy 76.2 147.32) (xy 97.79 147.32)
 		)
@@
 		)
 	)
-	(bus
-		(pts
-			(xy 124.46 59.69) (xy 124.46 62.23)
-		)
-		(stroke
-			(width 0)
-			(type default)
-		)
-	)
 	(wire
 		(pts
@@
 		)
 	)
-	(bus
-		(pts
-			(xy 124.46 62.23) (xy 124.46 64.77)
-		)
-		(stroke
-			(width 0)
-			(type default)
-		)
-	)
 	(wire
 		(pts
@@
 	(wire
 		(pts
-			(xy 127 59.69) (xy 148.59 59.69)
-		)
-		(stroke
-			(width 0)
-			(type default)
-		)
-	)
-	(wire
-		(pts
 			(xy 76.2 165.1) (xy 97.79 165.1)
 		)
@@
 	(bus
 		(pts
-			(xy 123.19 55.88) (xy 113.03 55.88)
-		)
-		(stroke
-			(width 0)
-			(type default)
-		)
-	)
-	(bus
-		(pts
 			(xy 72.39 128.27) (xy 62.23 128.27)
 		)
@@
 	(bus
 		(pts
-			(xy 123.19 55.88) (xy 124.46 57.15)
-		)
-		(stroke
-			(width 0)
-			(type default)
-		)
-	)
-	(bus
-		(pts
 			(xy 59.69 135.89) (xy 72.39 135.89)
 		)
@@
 		)
 	)
-	(bus
-		(pts
-			(xy 124.46 57.15) (xy 124.46 59.69)
-		)
-		(stroke
-			(width 0)
-			(type default)
-		)
-	)
 	(wire
 		(pts
@@
 		)
 	)
-	(wire
-		(pts
-			(xy 127 62.23) (xy 148.59 62.23)
-		)
-		(stroke
-			(width 0)
-			(type default)
-		)
-	)
 	(bus
 		(pts
@@
 	(wire
 		(pts
-			(xy 127 69.85) (xy 148.59 69.85)
-		)
-		(stroke
-			(width 0)
-			(type default)
-		)
-	)
-	(wire
-		(pts
 			(xy 134.62 149.86) (xy 113.03 149.86)
 		)
@@
 		(pts
 			(xy 73.66 129.54) (xy 72.39 128.27)
-		)
-		(stroke
-			(width 0)
-			(type default)
-		)
-	)
-	(bus
-		(pts
-			(xy 124.46 64.77) (xy 124.46 67.31)
 		)
 		(stroke
@@
 		)
 	)
-	(label "ADCDAC{ADCDAC}"
-		(at 113.03 55.88 0)
-		(fields_autoplaced yes)
-		(effects
-			(font
-				(size 1.27 1.27)
-			)
-			(justify left bottom)
-		)
-	)
 	(label "UART0.RX"
 		(at 134.62 119.38 180)
@@
 		)
 	)
-	(label "ADCDAC.HPOUTR"
-		(at 143.51 67.31 180)
-		(fields_autoplaced yes)
-		(effects
-			(font
-				(size 1.27 1.27)
-			)
-			(justify right bottom)
-		)
-	)
 	(label "LCD0{LCD_CTL}"
 		(at 36.83 26.67 0)
@@
 		)
 	)
-	(label "ADCDAC.HBIAS"
-		(at 143.51 69.85 180)
-		(fields_autoplaced yes)
-		(effects
-			(font
-				(size 1.27 1.27)
-			)
-			(justify right bottom)
-		)
-	)
 	(label "CSI.CSI_SDA"
 		(at 134.62 149.86 180)
@@
 		)
 	)
-	(label "ADCDAC.HPOUTL"
-		(at 143.51 64.77 180)
-		(fields_autoplaced yes)
-		(effects
-			(font
-				(size 1.27 1.27)
-			)
-			(justify right bottom)
-		)
-	)
 	(label "UART2{UART}"
 		(at 153.67 123.19 180)
@@
 		)
 	)
-	(label "ADCDAC.HPCOMFB"
-		(at 143.51 62.23 180)
-		(fields_autoplaced yes)
-		(effects
-			(font
-				(size 1.27 1.27)
-			)
-			(justify right bottom)
-		)
-	)
 	(label "LCD_D22"
 		(at 76.2 172.72 0)
@@
 		)
 	)
-	(label "ADCDAC.HPCOM"
-		(at 143.51 59.69 180)
-		(fields_autoplaced yes)
-		(effects
-			(font
-				(size 1.27 1.27)
-			)
-			(justify right bottom)
-		)
-	)

Commit message: pre production tests
Parts:
- J301: now not fitted; now left out of the parts list
Changed lines of the file:
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@@
 		(unit 1)
 		(exclude_from_sim no)
-		(in_bom yes)
+		(in_bom no)
 		(on_board yes)
-		(dnp no)
+		(dnp yes)
 		(fields_autoplaced yes)
 		(property "Reference" "J301"
